Commit message: Add files via upload

File: tribot/urdf/tribot_base.xacro (robot description, xacro)
@@ -3,5 +3,5 @@
     <xacro:macro name="tribot_base">
         <!-- base link 在地面的投影 -->
-        <link name="base_footprint">
+        <link name="${tf_prefix}base_footprint">
             <visual>
                 <origin xyz="0 0 0" rpy="0 0 0" />
@@ -11,14 +11,14 @@
             </visual>
         </link>
-        <gazebo reference="base_footprint">
+        <gazebo reference="${tf_prefix}base_footprint">
             <turnGravityOff>false</turnGravityOff>
         </gazebo>
         <joint name="base_footprint_joint" type="fixed">
             <origin xyz="0 0 0.01" rpy="0 0 0" />  <!-- 0.01m is the height of base...between the 2 frames -->
-            <parent link="base_footprint"/>
-            <child link="base_link" />
+            <parent link="${tf_prefix}base_footprint"/>
+            <child link="${tf_prefix}base_link" />
         </joint>
         <link
-            name="base_link">
+            name="${tf_prefix}base_link">
             <inertial>
             <origin
@@ -59,5 +59,5 @@
             </collision>
         </link>
-        <gazebo reference="base_link">
+        <gazebo reference="${tf_prefix}base_link">
             <material>Gazebo/White</material>
         </gazebo>

File: tribot/urdf/tribot_camera.xacro (robot description, xacro)
@@ -3,5 +3,5 @@
     <xacro:macro name="tribot_camera" params="prefix:=camera">
         <link
-            name="camera_link">
+            name="${tf_prefix}camera_link">
             <inertial>
             <origin
@@ -43,8 +43,8 @@
         </link>
         <!-- reference here must be the same with link name above -->
-        <gazebo reference="camera_link">
+        <gazebo reference="${tf_prefix}camera_link">
             <material>Gazebo/Red</material>
         </gazebo>
-        <gazebo reference="camera_link">
+        <gazebo reference="${tf_prefix}camera_link">
             <sensor type="depth" name="${prefix}">
                 <always_on>true</always_on>
@@ -67,10 +67,10 @@
                     <alwaysOn>true</alwaysOn>
                     <updateRate>10</updateRate>
-                    <imageTopicName>rgb/image_raw</imageTopicName>
-                    <depthImageTopicName>depth/image_raw</depthImageTopicName>
-                    <pointCloudTopicName>depth/points</pointCloudTopicName>
-                    <cameraInfoTopicName>rgb/camera_info</cameraInfoTopicName>
-                    <depthImageCameraInfoTopicName>depth/camera_info</depthImageCameraInfoTopicName>
-                    <frameName>camera_link</frameName>
+                    <imageTopicName>rgb/${tf_prefix}image_raw</imageTopicName>
+                    <depthImageTopicName>depth/${tf_prefix}image_raw</depthImageTopicName>
+                    <pointCloudTopicName>depth/${tf_prefix}points</pointCloudTopicName>
+                    <cameraInfoTopicName>rgb/${tf_prefix}camera_info</cameraInfoTopicName>
+                    <depthImageCameraInfoTopicName>depth/${tf_prefix}camera_info</depthImageCameraInfoTopicName>
+                    <frameName>${tf_prefix}camera_link</frameName>
                     <!-- the same name with reference="camera_link" -->
                     <baseline>0.1</baseline>

File: tribot/urdf/tribot_gazebo_follower.xacro (robot description, xacro)
@@ -2,5 +2,5 @@
 <robot name="tribot" xmlns:xacro="http://www.ros.org/wiki/xacro">
     <xacro:property name="M_PI" value="3.1415926"/>
-    <xacro:property name="tf_prefix" value="leader_tribot/"/>
+    <xacro:property name="tf_prefix" value="tribot1/"/>
     <xacro:include filename="$(find tribot)/urdf/tribot_base.xacro" />
     <xacro:tribot_base/>

File: tribot/urdf/tribot_lidar.xacro (robot description, xacro)
@@ -4,5 +4,5 @@
         <!-- Create laser reference frame -->
         <link
-            name="lidar_link">
+            name="${tf_prefix}lidar_link">
             <inertial>
             <origin
@@ -44,8 +44,8 @@
         </link>
         <!-- reference here must be the same with link name above -->
-        <gazebo reference="lidar_link">
+        <gazebo reference="${tf_prefix}lidar_link">
             <material>Gazebo/Black</material>
         </gazebo>
-        <gazebo reference="lidar_link">
+        <gazebo reference="${tf_prefix}lidar_link">
             <sensor type="ray" name="tribot_lidar">
                 <pose>0 0 0 0 0 0</pose>
@@ -74,6 +74,6 @@
                 <plugin name="gazebo_rplidar" filename="libgazebo_ros_laser.so">
                     <robotNamespace>/</robotNamespace>
-                    <topicName>/scan</topicName>
-                    <frameName>lidar_link</frameName>
+                    <topicName>/${tf_prefix}scan</topicName>
+                    <frameName>${tf_prefix}lidar_link</frameName>
                     <!-- the same name with reference="lidar_link" -->
                 </plugin>

File: tribot/urdf/tribot_wheel.xacro (robot description, xacro)
@@ -2,5 +2,5 @@
 <robot xmlns:xacro="http://www.ros.org/wiki/xacro" name="tribot_wheel">
     <xacro:macro name="tribot_wheel" params="prefix">
-        <gazebo reference="${prefix}_link">
+        <gazebo reference="${tf_prefix}${prefix}_link">
             <material>Gazebo/DarkGrey</material>
         </gazebo>
